File: kicad/shadok/shadok.sch (KiCad schematic (older format))
At the start: 12 parts, among them J101 Conn_01x07_Female, J102 GS3, J103 TEST_1P, J104 TEST_1P, J105 SERIALS, SW101 SW_Push, X101 KXO-V97 50MHz

Commit message: fixed the fuckups from the first version
had to remove video module
Changed lines of the file:
@@
 EESchema Schematic File Version 4
+LIBS:shadok-cache
 EELAYER 26 0
 EELAYER END
@@
 F7 "~RAS" I L 8500 2450 50
 F8 "~CAS" I L 8500 2550 50
+F9 "~ЗПЗУ" I L 8500 1950 50
+F10 "~ЧТЗУ" I L 8500 2050 50
+F11 "~ЧТВВ" I L 8500 2150 50
+F12 "~ЗПВВ" I L 8500 2250 50
+F13 "СТЕК" I L 8500 2650 50
 $EndSheet
 Text Label 10200 3150 0    47   ~ 0
@@
 Wire Bus Line
 	550  6850 6350 6850
+Text Label 8500 1950 2    47   ~ 0
+VIDEOBW
+Text Label 8500 2050 2    47   ~ 0
+HVSYNC
+Text Label 8500 2150 2    47   ~ 0
+ADC_SYNCp
+Text Label 8500 2250 2    47   ~ 0
+ADC_SYNCINT
+Text Label 8500 2650 2    47   ~ 0
+ADC_SYNCn
 $EndSCHEMATC
