File: kicad/shadok/videopass.sch (KiCad schematic (older format))
At the start: 24 parts, among them J901 Conn_02x04_Odd_Even, J913 DIN-5, Q901 BC817, Q902 BC807, Q903 BC817

Commit message: fixed the fuckups from the first version
had to remove video module
Parts:
- removed C901: 10.0, Capacitors_Tantalum_SMD:CP_Tantalum_Case-B_EIA-3528-21_Reflow, symbol device:CP1_Small
- removed C902: 220, Capacitors_SMD:C_0805, symbol device:C_Small
- removed C903, C906, C907: 0.1, Capacitors_SMD:C_0603, symbol device:C_Small
- removed C904: 33, Capacitors_SMD:C_0805, symbol device:C_Small
- removed C905: 68.0, Capacitors_Tantalum_SMD:CP_Tantalum_Case-D_EIA-7343-31_Reflow, symbol device:CP1_Small
- removed D901: BAT54S, TO_SOT_Packages_SMD:SOT-23, symbol diode:BAT54S
- removed J901: Conn_02x04_Odd_Even, Socket_Strips:Socket_Strip_Angled_2x04_Pitch2.54mm, symbol conn:Conn_02x04_Odd_Even
- removed J913: DIN-5, w_conn_av:din-5, symbol conn:DIN-5
- removed L901: LQH66SN101M 100uH, Resistors_SMD:R_0805, symbol device:L
- removed Q901, Q903: BC817, TO_SOT_Packages_SMD:SOT-23, symbol transistors:BC817
- removed Q902: BC807, TO_SOT_Packages_SMD:SOT-23, symbol transistors:BC807
- removed R901, R909: 75, Resistors_SMD:R_0805, symbol device:R
- removed R902: 220, Resistors_SMD:R_0805, symbol device:R
- removed R903, R907: 1K2, Resistors_SMD:R_0805, symbol device:R
- removed R904: 470, Resistors_SMD:R_0805, symbol device:R
- removed R905, R908: 1K, Resistors_SMD:R_0805, symbol device:R
- removed R906: 6K8, Resistors_SMD:R_0805, symbol device:R
- removed RV901: 100K, Potentiometers:Potentiometer_Bourns_3296W_3-8Zoll_Inline_ScrewUp, symbol device:POT
Connections:
- net labels removed: +2V5
- wire segments 72 -> 9
