File: kicad/shadok-cheap/anal.sch (KiCad schematic (older format))
At the start: 28 parts, among them J801 Conn_01x02, J815 Audio Out, U801 TPA6110A2

Commit message: version 2 with all the required signals
Parts:
- removed C812, C814: 5pF (N/C), Capacitors_SMD:C_0805, symbol device:C_Small
- C820, C821, C822: footprint Capacitors_Tantalum_SMD:CP_Tantalum_Case-D_EIA-7343-31_Reflow -> Capacitors_Tantalum_SMD:CP_Tantalum_Case-B_EIA-3528-21_Reflow
- R811, R814: value R -> 15K
Connections:
- wire segments 76 -> 69
Changed lines of the file:
@@
 $Descr A4 11693 8268
 encoding utf-8
-Sheet 8 9
+Sheet 8 8
 Title "Analog I/O"
 Date ""
@@
 P 7200 3950
 F 0 "R811" H 7130 3904 50  0000 R CNN
-F 1 "R" H 7130 3995 50  0000 R CNN
+F 1 "15K" H 7130 3995 50  0000 R CNN
 F 2 "Resistors_SMD:R_0805" V 7130 3950 50  0001 C CNN
 F 3 "" H 7200 3950 50  0001 C CNN
@@
 P 7800 3950
 F 0 "R814" H 7730 3904 50  0000 R CNN
-F 1 "R" H 7730 3995 50  0000 R CNN
+F 1 "15K" H 7730 3995 50  0000 R CNN
 F 2 "Resistors_SMD:R_0805" V 7730 3950 50  0001 C CNN
 F 3 "" H 7800 3950 50  0001 C CNN
@@
 F 0 "C821" H 8100 3300 50  0000 L CNN
 F 1 "68.0" H 8100 3200 50  0000 L CNN
-F 2 "Capacitors_Tantalum_SMD:CP_Tantalum_Case-D_EIA-7343-31_Reflow" H 8350 3200 50  0001 C CNN
+F 2 "Capacitors_Tantalum_SMD:CP_Tantalum_Case-B_EIA-3528-21_Reflow" H 8350 3200 50  0001 C CNN
 F 3 "" H 8350 3200 50  0001 C CNN
 	1    8350 3200
@@
 F 0 "C820" V 10000 4550 50  0000 C CNN
 F 1 "68.0" V 10000 4300 50  0000 C CNN
-F 2 "Capacitors_Tantalum_SMD:CP_Tantalum_Case-D_EIA-7343-31_Reflow" H 9850 4500 50  0001 C CNN
+F 2 "Capacitors_Tantalum_SMD:CP_Tantalum_Case-B_EIA-3528-21_Reflow" H 9850 4500 50  0001 C CNN
 F 3 "" H 9850 4500 50  0001 C CNN
 	1    9850 4500
@@
 F 0 "C822" V 9950 4650 50  0000 C CNN
 F 1 "68.0" V 9950 4450 50  0000 C CNN
-F 2 "Capacitors_Tantalum_SMD:CP_Tantalum_Case-D_EIA-7343-31_Reflow" H 10100 4600 50  0001 C CNN
+F 2 "Capacitors_Tantalum_SMD:CP_Tantalum_Case-B_EIA-3528-21_Reflow" H 10100 4600 50  0001 C CNN
 F 3 "" H 10100 4600 50  0001 C CNN
 	1    10100 4600
 	0    -1   -1   0
 $EndComp
-$Comp
-L device:C_Small C812
-U 1 1 5BD93726
-P 7450 3950
-F 0 "C812" H 7600 3450 50  0000 C CNN
-F 1 "5pF (N/C)" H 7450 3550 50  0000 C CNN
-F 2 "Capacitors_SMD:C_0805" H 7450 3950 50  0001 C CNN
-F 3 "" H 7450 3950 50  0001 C CNN
-	1    7450 3950
-	-1   0    0    1
-$EndComp
-Wire Wire Line
-	7200 4150 7450 4150
-Wire Wire Line
-	7450 4150 7450 4050
-Connection ~ 7200 4150
 Wire Wire Line
 	7200 4150 7200 4550
 Wire Wire Line
-	7450 3850 7450 3750
-Wire Wire Line
-	7450 3750 7200 3750
-Connection ~ 7200 3750
-Wire Wire Line
 	7200 3750 7200 3800
-$Comp
-L device:C_Small C814
-U 1 1 5BDA3FBC
-P 8050 3950
-F 0 "C814" H 8200 3450 50  0000 C CNN
-F 1 "5pF (N/C)" H 8050 3550 50  0000 C CNN
-F 2 "Capacitors_SMD:C_0805" H 8050 3950 50  0001 C CNN
-F 3 "" H 8050 3950 50  0001 C CNN
-	1    8050 3950
-	-1   0    0    1
-$EndComp
-Wire Wire Line
-	8050 3850 8050 3750
-Connection ~ 8050 3750
 Wire Wire Line
 	8050 3750 7800 3750
 Wire Wire Line
-	7800 4150 8050 4150
-Wire Wire Line
-	8050 4150 8050 4050
-Connection ~ 7800 4150
-Wire Wire Line
 	7800 4150 7800 4300

Commit message: first working version
kvaz in sdram
AY emulation
Parts:
- C820, C822: value 68.0 -> 47.0
- C821: value 68.0 -> 47.0; footprint Capacitors_Tantalum_SMD:CP_Tantalum_Case-B_EIA-3528-21_Reflow -> Capacitors_Tantalum_SMD:CP_Tantalum_Case-D_EIA-7343-31_Reflow
- L801: value LQH66SN101M 100uH -> BLM21AG102SN1D
Changed lines of the file:
@@
 P 8350 3200
 F 0 "C821" H 8100 3300 50  0000 L CNN
-F 1 "68.0" H 8100 3200 50  0000 L CNN
-F 2 "Capacitors_Tantalum_SMD:CP_Tantalum_Case-B_EIA-3528-21_Reflow" H 8350 3200 50  0001 C CNN
+F 1 "47.0" H 8100 3200 50  0000 L CNN
+F 2 "Capacitors_Tantalum_SMD:CP_Tantalum_Case-D_EIA-7343-31_Reflow" H 8350 3200 50  0001 C CNN
 F 3 "" H 8350 3200 50  0001 C CNN
 	1    8350 3200
@@
 P 9850 4500
 F 0 "C820" V 10000 4550 50  0000 C CNN
-F 1 "68.0" V 10000 4300 50  0000 C CNN
+F 1 "47.0" V 10000 4300 50  0000 C CNN
 F 2 "Capacitors_Tantalum_SMD:CP_Tantalum_Case-B_EIA-3528-21_Reflow" H 9850 4500 50  0001 C CNN
 F 3 "" H 9850 4500 50  0001 C CNN
@@
 P 10100 4600
 F 0 "C822" V 9950 4650 50  0000 C CNN
-F 1 "68.0" V 9950 4450 50  0000 C CNN
+F 1 "47.0" V 9950 4450 50  0000 C CNN
 F 2 "Capacitors_Tantalum_SMD:CP_Tantalum_Case-B_EIA-3528-21_Reflow" H 10100 4600 50  0001 C CNN
 F 3 "" H 10100 4600 50  0001 C CNN
@@
 P 8900 3100
 F 0 "L801" V 9090 3100 50  0000 C CNN
-F 1 "LQH66SN101M 100uH" V 8999 3100 50  0000 C CNN
+F 1 "BLM21AG102SN1D" V 8999 3100 50  0000 C CNN
 F 2 "Resistors_SMD:R_0805" H 8900 3100 50  0001 C CNN
 F 3 "" H 8900 3100 50  0001 C CNN

Commit message: schematic sheet update  + pdf
Connections:
- wire segments 69 -> 65
Changed lines of the file:
@@
 	9550 4500 9550 3750
-Wire Wire Line
-	9550 3750 8050 3750
 Wire Wire Line
 	7800 3750 7800 3800
@@
 Wire Wire Line
 	9700 3650 7200 3650
-Wire Wire Line
-	7200 3650 7200 3750
 Connection ~ 9700 4600
 Wire Wire Line
@@
 	-1   0    0    1
 $EndComp
-Wire Wire Line
-	7800 4100 7800 4150
 Connection ~ 7800 4300
 Wire Wire Line
 	7800 4300 8250 4300
-Wire Wire Line
-	7200 4100 7200 4150
 Connection ~ 7200 4550
 Wire Wire Line
@@
 	0    -1   -1   0
 $EndComp
-Wire Wire Line
-	7200 4150 7200 4550
-Wire Wire Line
-	7200 3750 7200 3800
-Wire Wire Line
-	8050 3750 7800 3750
-Wire Wire Line
-	7800 4150 7800 4300
 $Comp
 L device:R R804
@@
 Text Label 8800 5100 0    50   ~ 0
 POWERPAD
+Wire Wire Line
+	7800 3750 9550 3750
+Wire Wire Line
+	7200 3650 7200 3800
+Wire Wire Line
+	7800 4100 7800 4300
+Wire Wire Line
+	7200 4100 7200 4550
 $EndSCHEMATC
