File: kicad/shadok-cheap/shadok.sch (KiCad schematic (older format))
At the start: 9 parts, among them J101 TEST_1P, J103 TEST_1P, J104 TEST_1P, J105 SERIALS, SW101 SW_Push, X101 KXO-V97 50MHz

Commit message: first working version
kvaz in sdram
AY emulation
Parts:
- added R101, R103: 100, Resistors_SMD:R_0805, symbol device:R
Connections:
- net labels added: ~DDIR
- net labels removed: FREE_IO1
- wire segments 96 -> 98
Changed lines of the file:
@@
 F10 "SO" I R 10200 2750 50
 $EndSheet
-Text Label 10850 3450 0    47   ~ 0
+Text Label 11050 3150 0    47   ~ 0
 ESP_TxD
-Text Label 10850 3350 0    47   ~ 0
+Text Label 10850 2900 0    47   ~ 0
 ESP_RxD
 Text Label 6700 4250 0    47   ~ 0
@@
 F12 "~ЗПВВ" I L 8500 2250 50
 F13 "СТЕК" I L 8500 2650 50
+F14 "~DDIR" I L 8500 2800 50
 $EndSheet
 Text Label 10200 3150 0    47   ~ 0
@@
 NoConn ~ 1400 2450
 Text Label 1400 2750 2    47   ~ 0
-FREE_IO1
+~DDIR
 Text Label 1400 2850 2    47   ~ 0
 FREE_IO2
 Text Label 7300 950  2    47   ~ 0
-FREE_IO1
+~DDIR
 $Comp
 L conn:TEST_1P J101
@@
 Wire Wire Line
 	7450 950  7300 950
+$Comp
+L device:R R101
+U 1 1 5B429F86
+P 10850 3050
+F 0 "R101" V 10950 3000 50  0000 C CNN
+F 1 "100" V 10850 3050 50  0000 C CNN
+F 2 "Resistors_SMD:R_0805" V 10780 3050 50  0001 C CNN
+F 3 "" H 10850 3050 50  0001 C CNN
+	1    10850 3050
+	1    0    0    -1
+$EndComp
+$Comp
+L device:R R103
+U 1 1 5B42A0E1
+P 11050 3300
+F 0 "R103" V 11150 3250 50  0000 C CNN
+F 1 "100" V 11050 3300 50  0000 C CNN
+F 2 "Resistors_SMD:R_0805" V 10980 3300 50  0001 C CNN
+F 3 "" H 11050 3300 50  0001 C CNN
+	1    11050 3300
+	1    0    0    -1
+$EndComp
+Wire Wire Line
+	10850 3200 10850 3350
+Wire Wire Line
+	10850 3450 11050 3450
+Text Label 8500 2800 2    47   ~ 0
+~DDIR
 Wire Bus Line
 	1100 550  1100 1950

Commit message: schematic sheet update  + pdf
Other:
- note added: "BODGE IN REV1"
Changed lines of the file:
@@
 Text Label 8500 2800 2    47   ~ 0
 ~DDIR
+Text Notes 10850 2650 0    50   ~ 0
+BODGE IN REV1
+Wire Notes Line
+	11700 2750 10750 2750
+Wire Notes Line
+	10750 2750 10750 2950
+Wire Notes Line
+	11700 2750 11700 3000
+Text Notes 6450 800  0    50   ~ 0
+BODGE IN REV1
+Wire Notes Line
+	7100 900  7100 800
+Wire Notes Line
+	7100 800  6450 800
 Wire Bus Line
 	1100 550  1100 1950

Commit message: sdram arbitre for zpu or anything really WIP
Connections:
- net labels added: СБРОС
- net labels removed: FREE_I1
Changed lines of the file:
@@
 encoding utf-8
 Sheet 1 8
-Title "Les Shadoks для Вектора-06ц"
+Title "ЛЕШАДОК ПОМПЕ для Вектора-06ц"
 Date ""
-Rev ""
-Comp ""
+Rev "2"
+Comp "http://sensi.org/~~svo"
 Comment1 "Les Shadoks pompaient"
 Comment2 ""
@@
 Wire Wire Line
 	1050 3650 1400 3650
-Text Notes 7550 3100 0    28   ~ 0
+Text Notes 7400 3100 0    28   ~ 0
 MSEL=[0,1,0]: AS (EPCS4) 3.3V\nMSEL=[0,0,0]: PS (ESP12F) 3.3V
 Text Label 8600 4100 2    47   ~ 0
@@
 	1400 3050 1200 3050
 Wire Wire Line
-	6700 3050 7250 3050
+	6700 3050 7100 3050
 Text Label 10200 2950 0    47   ~ 0
 DCLK/SPICLK
@@
 	5800 6200 5800 6600
 $Sheet
-S 8500 1450 650  1550
+S 8500 1450 650  1600
 U 5A80A983
 F0 "BUS" 50
@@
 F13 "СТЕК" I L 8500 2650 50
 F14 "~DDIR" I L 8500 2800 50
+F15 "СБРОС" I L 8500 3000 50
 $EndSheet
 Text Label 10200 3150 0    47   ~ 0
@@
 $EndComp
 Text Label 650  4050 0    47   ~ 0
-FREE_I1
-Text Label 7300 1050 2    47   ~ 0
+СБРОС
+Text Label 7300 1200 2    47   ~ 0
 FREE_IO2
-Text Label 7300 1150 2    47   ~ 0
-FREE_I1
 $Comp
 L power:+3V3 #PWR05
@@
 BUTT1
 Wire Wire Line
-	7300 1050 7450 1050
+	7300 1200 7450 1200
 Wire Wire Line
-	7300 1150 7450 1150
+	7300 1050 7450 1050
 $Comp
 L conn:TEST_1P J103
 U 1 1 5A82FD6E
-P 7450 1050
-F 0 "J103" V 7404 1238 50  0000 L CNN
-F 1 "TEST_1P" V 7250 1050 50  0001 L CNN
-F 2 "wirepads:WIREPAD_SMD_TINY" H 7650 1050 50  0001 C CNN
-F 3 "" H 7650 1050 50  0001 C CNN
-	1    7450 1050
+P 7450 1200
+F 0 "J103" V 7404 1388 50  0000 L CNN
+F 1 "TEST_1P" V 7250 1200 50  0001 L CNN
+F 2 "wirepads:WIREPAD_SMD_TINY" H 7650 1200 50  0001 C CNN
+F 3 "" H 7650 1200 50  0001 C CNN
+	1    7450 1200
 	0    1    1    0
 $EndComp
@@
 L conn:TEST_1P J104
 U 1 1 5A82FDEF
-P 7450 1150
-F 0 "J104" V 7404 1338 50  0000 L CNN
-F 1 "TEST_1P" V 7550 1150 50  0001 L CNN
-F 2 "wirepads:WIREPAD_SMD_TINY" H 7650 1150 50  0001 C CNN
-F 3 "" H 7650 1150 50  0001 C CNN
-	1    7450 1150
+P 7450 1050
+F 0 "J104" V 7404 1238 50  0000 L CNN
+F 1 "TEST_1P" V 7550 1050 50  0001 L CNN
+F 2 "wirepads:WIREPAD_SMD_TINY" H 7650 1050 50  0001 C CNN
+F 3 "" H 7650 1050 50  0001 C CNN
+	1    7450 1050
 	0    1    1    0
 $EndComp
@@
 L power:GND #PWR0147
 U 1 1 5B4DD7CA
-P 7250 3050
-F 0 "#PWR0147" H 7250 2800 50  0001 C CNN
-F 1 "GND" V 7255 2922 50  0000 R CNN
-F 2 "" H 7250 3050 50  0001 C CNN
-F 3 "" H 7250 3050 50  0001 C CNN
-	1    7250 3050
+P 7100 3050
+F 0 "#PWR0147" H 7100 2800 50  0001 C CNN
+F 1 "GND" V 7105 2922 50  0000 R CNN
+F 2 "" H 7100 3050 50  0001 C CNN
+F 3 "" H 7100 3050 50  0001 C CNN
+	1    7100 3050
 	0    -1   -1   0
 $EndComp
@@
 Wire Notes Line
 	7100 800  6450 800
+Text Label 8500 3000 2    47   ~ 0
+СБРОС
+Text Label 7300 1050 2    47   ~ 0
+СБРОС
+Wire Notes Line
+	7000 1000 6900 1000
+Wire Notes Line
+	6900 1000 6900 800
 Wire Bus Line
 	1100 550  1100 1950

Commit message: documented bodge pulldown R502 across RN502
Connections:
- wire segments 98 -> 99
Changed lines of the file:
@@
 Text Label 1400 2650 2    47   ~ 0
 ~STATUS
-Text Label 1400 3150 2    47   ~ 0
+Text Label 1150 3150 0    47   ~ 0
 ~CONFIG
 Text Label 8600 4550 2    47   ~ 0
@@
 Wire Notes Line
 	6900 1000 6900 800
+Wire Wire Line
+	1150 3150 1400 3150
 Wire Bus Line
 	1100 550  1100 1950
