File: kicad/shadok-cheap/esp12f.sch (KiCad schematic (older format))
At the start: 11 parts, among them J501 Micro_SD_Card, J502 TEST_1P, U501 ESP12F

Commit message: documented bodge pulldown R502 across RN502
Parts:
- added R502: 4K7, Resistors_SMD:R_0603, symbol device:R
Connections:
- wire segments 51 -> 57
Other:
- note added: "10K pulldown on GPIO15\nshould be enough, but \nsomehow it isn't.\nBodge R502 to enable boot."
Changed lines of the file:
@@
 U 1 1 5B545FB5
 P 9450 3150
-F 0 "JP501" V 9404 3276 50  0000 L CNN
-F 1 "SERIAL BUTTLOAD" V 9495 3276 50  0000 L CNN
+F 0 "JP501" V 9500 3300 50  0000 L CNN
+F 1 "SERIAL BUTTLOAD" V 9600 3300 50  0000 L CNN
 F 2 "Pin_Headers:Pin_Header_Straight_1x02" H 9450 3150 50  0001 C CNN
 F 3 "" H 9450 3150 50  0001 C CNN
@@
 U 1 1 5ABFDCB1
 P 9900 2650
-F 0 "RN502" V 10150 2800 50  0000 C CNN
-F 1 "10K" V 10150 2550 50  0000 C CNN
+F 0 "RN502" V 9550 2600 50  0000 C CNN
+F 1 "10K" V 9550 2350 50  0000 C CNN
 F 2 "Resistors_SMD:R_Array_Concave_4x0603" V 10175 2650 50  0001 C CNN
 F 3 "" H 9900 2650 50  0001 C CNN
@@
 	9500 2650 9500 2750
 Wire Wire Line
-	9500 2750 9700 2750
+	9500 2750 9600 2750
 $Comp
 L power:GND #PWR018
@@
 $EndComp
 Wire Wire Line
-	10100 2750 10300 2750
+	10100 2750 10150 2750
 Wire Wire Line
 	8650 2650 9500 2650
+$Comp
+L device:R R502
+U 1 1 5B622777
+P 9900 2950
+F 0 "R502" V 9800 2950 50  0000 C CNN
+F 1 "4K7" V 9900 2950 50  0000 C CNN
+F 2 "Resistors_SMD:R_0603" V 9830 2950 50  0001 C CNN
+F 3 "" H 9900 2950 50  0001 C CNN
+	1    9900 2950
+	0    -1   -1   0
+$EndComp
+Wire Wire Line
+	9750 2950 9600 2950
+Wire Wire Line
+	9600 2950 9600 2750
+Connection ~ 9600 2750
+Wire Wire Line
+	9600 2750 9700 2750
+Wire Wire Line
+	10050 2950 10150 2950
+Wire Wire Line
+	10150 2950 10150 2750
+Connection ~ 10150 2750
+Wire Wire Line
+	10150 2750 10300 2750
+Text Notes 10150 3200 0    50   ~ 0
+10K pulldown on GPIO15\nshould be enough, but \nsomehow it isn't.\nBodge R502 to enable boot.
 $EndSCHEMATC

Commit message: verilog parts supplementing the last commit
Parts:
- RN502: value 10K -> 3K3
Other:
- note added: "10K pulldown on GPIO15\nshould be enough, but \nsomehow it isn't.\nIf RN502=10K, bodge \nR502 to enable boot."
- note removed: "10K pulldown on GPIO15\nshould be enough, but \nsomehow it isn't.\nBodge R502 to enable boot."
Changed lines of the file:
@@
 P 9900 2650
 F 0 "RN502" V 9550 2600 50  0000 C CNN
-F 1 "10K" V 9550 2350 50  0000 C CNN
+F 1 "3K3" V 9550 2350 50  0000 C CNN
 F 2 "Resistors_SMD:R_Array_Concave_4x0603" V 10175 2650 50  0001 C CNN
 F 3 "" H 9900 2650 50  0001 C CNN
@@
 Wire Wire Line
 	10150 2750 10300 2750
-Text Notes 10150 3200 0    50   ~ 0
-10K pulldown on GPIO15\nshould be enough, but \nsomehow it isn't.\nBodge R502 to enable boot.
+Text Notes 10200 3250 0    50   ~ 0
+10K pulldown on GPIO15\nshould be enough, but \nsomehow it isn't.\nIf RN502=10K, bodge \nR502 to enable boot.
 $EndSCHEMATC
