File: kicad/shadok-cheap/bus.sch (KiCad schematic (older format))
At the start: 15 parts, among them J601 74LVC8T245, J602 74LVC8T245, J603 74LVC8T245, J604 SNP34-90, J605 74LVC8T245, U601 74LVC1T45

Commit message: first working version
kvaz in sdram
AY emulation
Connections:
- net labels added: ~DDIR
- wire segments 298 -> 294
Changed lines of the file:
@@
 Connection ~ 9500 850
-Wire Wire Line
-	9500 850  9800 850
 Wire Wire Line
 	8600 1050 8900 1050
@@
 	9200 1050 9500 1050
 Connection ~ 9500 1050
-Wire Wire Line
-	9500 1050 9800 1050
 $Comp
 L power:GND #PWR0626
@@
 	1    0    0    -1
 $EndComp
-Wire Wire Line
-	9800 850  10100 850
-Wire Wire Line
-	9800 1050 10100 1050
 $Comp
 L device:C_Small C602
@@
 	9200 1450 9500 1450
 Connection ~ 9500 1450
-Wire Wire Line
-	9500 1450 9800 1450
-Wire Wire Line
-	9800 1450 10100 1450
-Wire Wire Line
-	10100 1650 9800 1650
 Connection ~ 8900 1650
 Wire Wire Line
@@
 Wire Wire Line
 	9500 1650 9200 1650
-Wire Wire Line
-	9800 1650 9500 1650
 Text Notes 7250 6900 0    157  ~ 0
 Шинные приемопередатчики
 Text Label 9850 4850 0    47   ~ 0
-~БЛК
-Text Label 3900 4700 0    47   ~ 0
 ~БЛК
 Connection ~ 5900 5150
@@
 Wire Wire Line
 	10000 3650 10250 3650
-Wire Bus Line
-	5250 3650 5250 4350
-Wire Bus Line
-	1600 1150 1600 1850
-Wire Bus Line
-	1600 2900 1600 3600
-Wire Bus Line
-	4300 4350 4300 5550
-Wire Bus Line
-	1500 4850 1500 5650
 Text HLabel 10250 3350 2    50   Input ~ 0
 ~ЧТЗУ
@@
 Text HLabel 10250 3650 2    50   Input ~ 0
 СТЕК
+Wire Wire Line
+	9500 850  10100 850
+Wire Wire Line
+	9500 1050 10100 1050
+Wire Wire Line
+	9500 1450 10100 1450
+Wire Wire Line
+	9500 1650 10100 1650
+Wire Bus Line
+	5250 3650 5250 4350
+Wire Bus Line
+	1600 1150 1600 1850
+Wire Bus Line
+	1600 2900 1600 3600
+Wire Bus Line
+	4300 4350 4300 5550
+Wire Bus Line
+	1500 4850 1500 5650
+Text HLabel 3900 4700 2    50   Input ~ 0
+~DDIR
 $EndSCHEMATC

Commit message: sdram arbitre for zpu or anything really WIP
Parts:
- added Q?: BC817, TO_SOT_Packages_SMD:SOT-23, symbol transistors:BC817
- added R? (x2): 10K, Resistors_SMD:R_0805, symbol device:R
Connections:
- net labels added: СБРОС
- wire segments 294 -> 296
Other:
- note added: "BODGE IN REV 1"
Changed lines of the file:
@@
 Wire Wire Line
 	9500 1650 10100 1650
+Text HLabel 3900 4700 2    50   Input ~ 0
+~DDIR
+$Comp
+L transistors:BC817 Q?
+U 1 1 5B4E5996
+P 9150 6050
+F 0 "Q?" H 9341 6096 50  0000 L CNN
+F 1 "BC817" H 9341 6005 50  0000 L CNN
+F 2 "TO_SOT_Packages_SMD:SOT-23" H 9350 5975 50  0001 L CIN
+F 3 "http://www.fairchildsemi.com/ds/BC/BC817.pdf" H 9150 6050 50  0001 L CNN
+	1    9150 6050
+	1    0    0    -1
+$EndComp
+$Comp
+L device:R R?
+U 1 1 5B4E92C7
+P 8800 6050
+F 0 "R?" V 8900 6000 50  0000 C CNN
+F 1 "10K" V 8800 6050 50  0000 C CNN
+F 2 "Resistors_SMD:R_0805" V 8730 6050 50  0001 C CNN
+F 3 "" H 8800 6050 50  0001 C CNN
+	1    8800 6050
+	0    1    1    0
+$EndComp
+$Comp
+L device:R R?
+U 1 1 5B51308C
+P 9250 5700
+F 0 "R?" V 9350 5650 50  0000 C CNN
+F 1 "10K" V 9250 5700 50  0000 C CNN
+F 2 "Resistors_SMD:R_0805" V 9180 5700 50  0001 C CNN
+F 3 "" H 9250 5700 50  0001 C CNN
+	1    9250 5700
+	-1   0    0    1
+$EndComp
+$Comp
+L power:+3V3 #PWR?
+U 1 1 5B5130EE
+P 9250 5550
+F 0 "#PWR?" H 9250 5400 50  0001 C CNN
+F 1 "+3V3" H 9265 5723 50  0000 C CNN
+F 2 "" H 9250 5550 50  0001 C CNN
+F 3 "" H 9250 5550 50  0001 C CNN
+	1    9250 5550
+	1    0    0    -1
+$EndComp
+$Comp
+L power:GND #PWR?
+U 1 1 5B53CE61
+P 9250 6250
+F 0 "#PWR?" H 9250 6000 50  0001 C CNN
+F 1 "GND" H 9255 6077 50  0000 C CNN
+F 2 "" H 9250 6250 50  0001 C CNN
+F 3 "" H 9250 6250 50  0001 C CNN
+	1    9250 6250
+	1    0    0    -1
+$EndComp
+Wire Wire Line
+	7950 6050 8650 6050
+Text Label 7950 6050 0    50   ~ 0
+~СБРОСЪ
+Wire Wire Line
+	9250 5850 10100 5850
+Connection ~ 9250 5850
+Text HLabel 10100 5850 2    50   Input ~ 0
+СБРОС
+Wire Notes Line
+	8600 5300 8600 6500
+Wire Notes Line
+	8600 6500 10500 6500
+Wire Notes Line
+	10500 6500 10500 5300
+Wire Notes Line
+	10500 5300 8600 5300
 Wire Bus Line
 	5250 3650 5250 4350
@@
 Wire Bus Line
 	1500 4850 1500 5650
-Text HLabel 3900 4700 2    50   Input ~ 0
-~DDIR
+Text Notes 9750 6450 0    50   ~ 0
+BODGE IN REV 1
 $EndSCHEMATC

Commit message: documented bodge pulldown R502 across RN502
Parts:
- gave numbers to parts that had none: 3
Changed lines of the file:
@@
 ~DDIR
 $Comp
-L transistors:BC817 Q?
+L transistors:BC817 Q601
 U 1 1 5B4E5996
 P 9150 6050
-F 0 "Q?" H 9341 6096 50  0000 L CNN
+F 0 "Q601" H 9341 6096 50  0000 L CNN
 F 1 "BC817" H 9341 6005 50  0000 L CNN
 F 2 "TO_SOT_Packages_SMD:SOT-23" H 9350 5975 50  0001 L CIN
@@
 $EndComp
 $Comp
-L device:R R?
+L device:R R601
 U 1 1 5B4E92C7
 P 8800 6050
-F 0 "R?" V 8900 6000 50  0000 C CNN
+F 0 "R601" V 8900 6000 50  0000 C CNN
 F 1 "10K" V 8800 6050 50  0000 C CNN
 F 2 "Resistors_SMD:R_0805" V 8730 6050 50  0001 C CNN
@@
 $EndComp
 $Comp
-L device:R R?
+L device:R R602
 U 1 1 5B51308C
 P 9250 5700
-F 0 "R?" V 9350 5650 50  0000 C CNN
+F 0 "R602" V 9350 5650 50  0000 C CNN
 F 1 "10K" V 9250 5700 50  0000 C CNN
 F 2 "Resistors_SMD:R_0805" V 9180 5700 50  0001 C CNN
@@
 $EndComp
 $Comp
-L power:+3V3 #PWR?
+L power:+3V3 #PWR0632
 U 1 1 5B5130EE
 P 9250 5550
-F 0 "#PWR?" H 9250 5400 50  0001 C CNN
+F 0 "#PWR0632" H 9250 5400 50  0001 C CNN
 F 1 "+3V3" H 9265 5723 50  0000 C CNN
 F 2 "" H 9250 5550 50  0001 C CNN
@@
 $EndComp
 $Comp
-L power:GND #PWR?
+L power:GND #PWR0633
 U 1 1 5B53CE61
 P 9250 6250
-F 0 "#PWR?" H 9250 6000 50  0001 C CNN
+F 0 "#PWR0633" H 9250 6000 50  0001 C CNN
 F 1 "GND" H 9255 6077 50  0000 C CNN
 F 2 "" H 9250 6250 50  0001 C CNN

Commit message: joystick "C" on ports 2e/2f works well
Connections:
- wire segments 296 -> 299
- no-connect marks 8 -> 6
Changed lines of the file:
@@
 Text Label 7800 4850 2    50   ~ 0
 ~БЛКЪ
-Text Label 7850 4950 2    50   ~ 0
+Text Label 7950 4950 2    50   ~ 0
 ~ВВОДЪ_СИСТЕМЫ
 Text Label 7450 5050 2    50   ~ 0
@@
 	7100 4950 7950 4950
 NoConn ~ 7100 4650
-NoConn ~ 7100 4950
 NoConn ~ 7100 5150
-NoConn ~ 5900 4950
 NoConn ~ 5900 5150
 $Comp
@@
 Wire Wire Line
 	7950 6050 8650 6050
-Text Label 7950 6050 0    50   ~ 0
-~СБРОСЪ
 Wire Wire Line
 	9250 5850 10100 5850
@@
 Text Notes 9750 6450 0    50   ~ 0
 BODGE IN REV 1
+Text Label 7950 6050 0    50   ~ 0
+~ВВОДЪ_СИСТЕМЫ
+Wire Wire Line
+	7100 4950 7100 5000
+Wire Wire Line
+	7100 5000 5900 5000
+Wire Wire Line
+	5900 5000 5900 4950
 Wire Bus Line
 	5250 3650 5250 4350
@@
 Wire Bus Line
 	1500 4850 1500 5650
+Connection ~ 7100 4950
 $EndSCHEMATC
